File: Nucleo2USB.kicad_pcb (KiCad board)
At the start: 2 copper layers, 70 x 53 mm, 46 parts, among them U1 LM3526L, U3 ESDAxxSC6, U4 ESDAxxSC6, U5 MAX40200AUK, U6 MAX40200AUK, U7 MAX40200AUK, X1 USB-OTG, X2 USB-OTG, X3 ST-MORPHO-CN7, X4 ST-MORPHO-CN10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

Commit message: update pcb, add cache library
Parts:
- moved R17 6.36 mm to (134.7, 126.9)
- moved R18 6.36 mm to (136.1, 126.9)
- moved R20 4.37 mm to (135.4, 124.8), turned to 0 degrees
- moved X5 2.76 mm to (139.0, 124.5), turned to 90 degrees
Routing:
- net OTGHS_DN: track 63.6 -> 55.8 mm
- net OTGHS_DP: track 62.9 -> 55.9 mm
- net PA12: track 15.8 -> 20.9 mm
- net +3V3: track 63.3 -> 60.5 mm
- net PA11: track 18.9 -> 19.8 mm
